File: hardware/picodrone_controller/picodrone_controller.kicad_pcb (KiCad board)
At the start: 2 copper layers, 35.6 x 71.1 mm, 32 parts, among them J1 RPi Pico, J2 RPi Pico, J3 MPU6050, J4 SD Card, J5 Motor, J6 Motor, J7 Motor, J8 Motor, J9 Battery, Q1 NMOS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

Commit message: generated gerbers and ordered
Routing:
- net GND: track 16.3 -> 18.1 mm
- net VCC: track 14.5 -> 15.9 mm
Other:
- board text added: "PicoDrone Controller"
